File: BeaconBuddy.sch (KiCad schematic (older format))
At the start: 30 parts, among them P1 CONN_01X06, P2 AIN0, Q1 Si2365EDS, U1 nRF52832-QFAA, U3 BME280, Y1 32.768kHz, Y2 32MHz

Commit message: Add reset switch, second LED
Parts:
- added B?: SKRPABE010, symbol Button_SKRP
- added D?: L0603R, LEDs:LED_0603, symbol Led_Small
- added R?: 470, Resistors_SMD:R_0603, symbol R
Connections:
- net GND: no longer R1.2
- net VDD: now also R1.2, R?.2
- net at U1.19 (P0.16/TDATA[1]): now also D?.1 (K)
- net at U1.20 (P0.17): now also D1.1 (K); no longer D1.2 (A)
- net at R1.1: now also D1.2 (A); no longer D1.1 (K)
- new net: D?.2 (A), R?.1
Other:
- moved on the sheet: C1, D1
Changed lines of the file:
@@
 	7800 1300 7800 1400
 Wire Wire Line
-	4350 2700 4550 2700
+	3850 2700 4550 2700
 Wire Wire Line
 	6550 2700 7150 2700
@@
 $EndComp
 Wire Wire Line
-	4350 2700 4350 2550
-Wire Wire Line
-	4350 2550 4000 2550
-Wire Wire Line
-	4000 2550 4000 2700
+	3850 2700 3850 2850
 $Comp
 L C C1
 U 1 1 578479F3
-P 4000 2850
-F 0 "C1" H 4025 2950 50  0000 L CNN
-F 1 "0.1uF" H 4025 2750 50  0000 L CNN
-F 2 "Capacitors_SMD:C_0603" H 4038 2700 50  0001 C CNN
-F 3 "" H 4000 2850 50  0000 C CNN
-	1    4000 2850
-	1    0    0    -1
-$EndComp
-Wire Wire Line
-	4000 3000 4000 3100
+P 3850 3000
+F 0 "C1" H 3875 3100 50  0000 L CNN
+F 1 "0.1uF" H 3875 2900 50  0000 L CNN
+F 2 "Capacitors_SMD:C_0603" H 3888 2850 50  0001 C CNN
+F 3 "" H 3850 3000 50  0000 C CNN
+	1    3850 3000
+	1    0    0    -1
+$EndComp
+Wire Wire Line
+	3850 3150 3850 3250
 $Comp
 L GND #PWR16
 U 1 1 57847ADB
-P 4000 3100
-F 0 "#PWR16" H 4000 2850 50  0001 C CNN
-F 1 "GND" H 4000 2950 50  0000 C CNN
-F 2 "" H 4000 3100 50  0000 C CNN
-F 3 "" H 4000 3100 50  0000 C CNN
-	1    4000 3100
+P 3850 3250
+F 0 "#PWR16" H 3850 3000 50  0001 C CNN
+F 1 "GND" H 3850 3100 50  0000 C CNN
+F 2 "" H 3850 3250 50  0000 C CNN
+F 3 "" H 3850 3250 50  0000 C CNN
+	1    3850 3250
 	1    0    0    -1
 $EndComp
@@
 F 3 "" V 3850 4650 50  0000 C CNN
 	1    3850 4650
-	0    -1   -1   0
+	0    1    1    0
 $EndComp
 $Comp
@@
 Wire Wire Line
 	3850 5150 3850 5250
-$Comp
-L GND #PWR14
-U 1 1 5784817B
-P 3850 5250
-F 0 "#PWR14" H 3850 5000 50  0001 C CNN
-F 1 "GND" H 3850 5100 50  0000 C CNN
-F 2 "" H 3850 5250 50  0000 C CNN
-F 3 "" H 3850 5250 50  0000 C CNN
-	1    3850 5250
-	1    0    0    -1
-$EndComp
 $Comp
 L Battery BT1
@@
 Wire Wire Line
 	4000 1150 4050 1150
+$Comp
+L Button_SKRP B?
+U 1 1 580CED08
+P 2500 3900
+F 0 "B?" H 2500 4250 60  0000 C CNN
+F 1 "SKRPABE010" H 2500 3600 60  0000 C CNN
+F 2 "" H 2500 4000 60  0000 C CNN
+F 3 "" H 2500 4000 60  0000 C CNN
+	1    2500 3900
+	1    0    0    -1
+$EndComp
+$Comp
+L Led_Small D?
+U 1 1 580CF511
+P 3400 4650
+F 0 "D?" V 3400 4500 50  0000 L CNN
+F 1 "L0603R" V 3300 4300 50  0000 L CNN
+F 2 "LEDs:LED_0603" V 3400 4650 50  0001 C CNN
+F 3 "" V 3400 4650 50  0000 C CNN
+	1    3400 4650
+	0    1    1    0
+$EndComp
+$Comp
+L R R?
+U 1 1 580CF517
+P 3400 5000
+F 0 "R?" H 3500 5050 50  0000 C CNN
+F 1 "470" H 3500 4950 50  0000 C CNN
+F 2 "Resistors_SMD:R_0603" V 3330 5000 30  0001 C CNN
+F 3 "" H 3400 5000 30  0000 C CNN
+	1    3400 5000
+	1    0    0    -1
+$EndComp
+Wire Wire Line
+	3400 4400 4550 4400
+Wire Wire Line
+	3400 4400 3400 4550
+Wire Wire Line
+	3400 4750 3400 4850
+Wire Wire Line
+	3400 5150 3400 5250
+$Comp
+L VDD #PWR?
+U 1 1 580D18D1
+P 3850 5250
+F 0 "#PWR?" H 3850 5100 50  0001 C CNN
+F 1 "VDD" H 3850 5400 50  0000 C CNN
+F 2 "" H 3850 5250 50  0000 C CNN
+F 3 "" H 3850 5250 50  0000 C CNN
+	1    3850 5250
+	-1   0    0    1
+$EndComp
+$Comp
+L VDD #PWR?
+U 1 1 580D1B2E
+P 3400 5250
+F 0 "#PWR?" H 3400 5100 50  0001 C CNN
+F 1 "VDD" H 3400 5400 50  0000 C CNN
+F 2 "" H 3400 5250 50  0000 C CNN
+F 3 "" H 3400 5250 50  0000 C CNN
+	1    3400 5250
+	-1   0    0    1
+$EndComp
 $EndSCHEMATC

Commit message: Update PCB for rev.C
Parts:
- added R5: 10k, Resistors_SMD:R_0603, symbol R
- B1: renamed from B?; footprint (none) -> New_Footprints:SKRPABE010
- gave numbers to parts that had none: 2
Connections:
- net GND: now also B1.3
- net VDD: now also R5.1
- net nRESET: now also B1.1, R5.2
Other:
- moved on the sheet: B1, C14, C15, P1, P2, R2, R3, U3
